Commit message: feat: environment is completed

File: src/op3_description/urdf/robot.urdf (robot description, URDF)
Before this commit: robot robotis_op3, 25 links, 24 joints
Links:
- link body_link: geometry collision mesh filename=file:///home/lexciese/Dev/altair_gazebo_simulation/install/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 scale=0.001 0.001 0.001; visual mesh filename=file:///home/lexciese/Dev/altair_gazebo_simulation/install/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 scale=0.001 0.001 0.001
- link head_pan_link: geometry collision mesh filename=file:///home/lexciese/Dev/altair_gazebo_simulation/install/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 scale=0.001 0.001 0.001; visual mesh filename=file:///home/lexciese/Dev/altair_gazebo_simulation/install/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 scale=0.001 0.001 0.001
- link head_tilt_link: geometry collision mesh filename=file:///home/lexciese/Dev/altair_gazebo_simulation/install/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 scale=0.001 0.001 0.001; visual mesh filename=file:///home/lexciese/Dev/altair_gazebo_simulation/install/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 scale=0.001 0.001 0.001
- link l_ank_pitch_link: geometry collision mesh filename=file:///home/lexciese/Dev/altair_gazebo_simulation/install/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 scale=0.001 0.001 0.001; visual mesh filename=file:///home/lexciese/Dev/altair_gazebo_simulation/install/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 scale=0.001 0.001 0.001
- link l_ank_roll_link: geometry collision mesh filename=file:///home/lexciese/Dev/altair_gazebo_simulation/install/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 scale=0.001 0.001 0.001; visual mesh filename=file:///home/lexciese/Dev/altair_gazebo_simulation/install/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 scale=0.001 0.001 0.001
- link l_el_link: geometry collision mesh filename=file:///home/lexciese/Dev/altair_gazebo_simulation/install/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 scale=0.001 0.001 0.001; visual mesh filename=file:///home/lexciese/Dev/altair_gazebo_simulation/install/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 scale=0.001 0.001 0.001
- link l_hip_pitch_link: geometry collision mesh filename=file:///home/lexciese/Dev/altair_gazebo_simulation/install/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 scale=0.001 0.001 0.001; visual mesh filename=file:///home/lexciese/Dev/altair_gazebo_simulation/install/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 scale=0.001 0.001 0.001
- link l_hip_roll_link: geometry collision mesh filename=file:///home/lexciese/Dev/altair_gazebo_simulation/install/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 scale=0.001 0.001 0.001; visual mesh filename=file:///home/lexciese/Dev/altair_gazebo_simulation/install/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 scale=0.001 0.001 0.001
- link l_hip_yaw_link: geometry collision mesh filename=file:///home/lexciese/Dev/altair_gazebo_simulation/install/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 scale=0.001 0.001 0.001; visual mesh filename=file:///home/lexciese/Dev/altair_gazebo_simulation/install/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 scale=0.001 0.001 0.001
- link l_knee_link: geometry collision mesh filename=file:///home/lexciese/Dev/altair_gazebo_simulation/install/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 scale=0.001 0.001 0.001; visual mesh filename=file:///home/lexciese/Dev/altair_gazebo_simulation/install/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 scale=0.001 0.001 0.001
- link l_sho_pitch_link: geometry collision mesh filename=file:///home/lexciese/Dev/altair_gazebo_simulation/install/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 scale=0.001 0.001 0.001; visual mesh filename=file:///home/lexciese/Dev/altair_gazebo_simulation/install/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 scale=0.001 0.001 0.001
- link l_sho_roll_link: geometry collision mesh filename=file:///home/lexciese/Dev/altair_gazebo_simulation/install/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 scale=0.001 0.001 0.001; visual mesh filename=file:///home/lexciese/Dev/altair_gazebo_simulation/install/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 scale=0.001 0.001 0.001
- link r_ank_pitch_link: geometry collision mesh filename=file:///home/lexciese/Dev/altair_gazebo_simulation/install/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 scale=0.001 0.001 0.001; visual mesh filename=file:///home/lexciese/Dev/altair_gazebo_simulation/install/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 scale=0.001 0.001 0.001
- link r_ank_roll_link: geometry collision mesh filename=file:///home/lexciese/Dev/altair_gazebo_simulation/install/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 scale=0.001 0.001 0.001; visual mesh filename=file:///home/lexciese/Dev/altair_gazebo_simulation/install/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 scale=0.001 0.001 0.001
- link r_el_link: geometry collision mesh filename=file:///home/lexciese/Dev/altair_gazebo_simulation/install/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 scale=0.001 0.001 0.001; visual mesh filename=file:///home/lexciese/Dev/altair_gazebo_simulation/install/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 scale=0.001 0.001 0.001
- link r_hip_pitch_link: geometry collision mesh filename=file:///home/lexciese/Dev/altair_gazebo_simulation/install/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 scale=0.001 0.001 0.001; visual mesh filename=file:///home/lexciese/Dev/altair_gazebo_simulation/install/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 scale=0.001 0.001 0.001
- link r_hip_roll_link: geometry collision mesh filename=file:///home/lexciese/Dev/altair_gazebo_simulation/install/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 scale=0.001 0.001 0.001; visual mesh filename=file:///home/lexciese/Dev/altair_gazebo_simulation/install/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 scale=0.001 0.001 0.001
- link r_hip_yaw_link: geometry collision mesh filename=file:///home/lexciese/Dev/altair_gazebo_simulation/install/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 scale=0.001 0.001 0.001; visual mesh filename=file:///home/lexciese/Dev/altair_gazebo_simulation/install/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 scale=0.001 0.001 0.001
- link r_knee_link: geometry collision mesh filename=file:///home/lexciese/Dev/altair_gazebo_simulation/install/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 scale=0.001 0.001 0.001; visual mesh filename=file:///home/lexciese/Dev/altair_gazebo_simulation/install/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 scale=0.001 0.001 0.001
- link r_sho_pitch_link: geometry collision mesh filename=file:///home/lexciese/Dev/altair_gazebo_simulation/install/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 scale=0.001 0.001 0.001; visual mesh filename=file:///home/lexciese/Dev/altair_gazebo_simulation/install/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 scale=0.001 0.001 0.001
- link r_sho_roll_link: geometry collision mesh filename=file:///home/lexciese/Dev/altair_gazebo_simulation/install/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 scale=0.001 0.001 0.001; visual mesh filename=file:///home/lexciese/Dev/altair_gazebo_simulation/install/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 scale=0.001 0.001 0.001

File: src/op3_description/urdf/robotis_op3.gazebo.xacro (robot description, xacro)
@@ -1,39 +1,26 @@
 <?xml version="1.0"?>
 <robot xmlns:xacro="http://ros.org/wiki/xacro">
-  <plugin name="gazebo_ros_joint_state_publisher"
-          filename="libgazebo_ros_joint_state_publisher.so">
-    <update_rate>20</update_rate>
-    <joint_name>l_hip_yaw</joint_name>
-    <joint_name>l_hip_roll</joint_name>
-    <joint_name>l_hip_pitch</joint_name>
-    <joint_name>l_knee</joint_name>
-    <joint_name>l_ank_roll</joint_name>
-    <joint_name>l_ank_pitch</joint_name>
-    <joint_name>r_hip_yaw</joint_name>
-    <joint_name>r_hip_roll</joint_name>
-    <joint_name>r_hip_pitch</joint_name>
-    <joint_name>r_knee</joint_name>
-    <joint_name>r_ank_roll</joint_name>
-    <joint_name>r_ank_pitch</joint_name>
-    <joint_name>l_sho_pitch</joint_name>
-    <joint_name>l_sho_roll</joint_name>
-    <joint_name>l_el</joint_name>
-    <joint_name>r_sho_pitch</joint_name>
-    <joint_name>r_sho_roll</joint_name>
-    <joint_name>r_el</joint_name>
-    <joint_name>head_pan</joint_name>
-    <joint_name>head_tilt</joint_name>
+  <plugin filename="gz-sim-sensors-system"
+    name="gz::sim::systems::Sensors">
+    <render_engine>ogre2</render_engine>
   </plugin>
-  <gazebo>
-    <plugin name="gazebo_ros_joint_pose_trajectory"
-        filename="libgazebo_ros_joint_pose_trajectory.so">
-        <update_rate>20</update_rate>
-    </plugin>
-  </gazebo>
+  <plugin filename="gz-sim-imu-system"
+    name="gz::sim::systems::Imu">
+  </plugin>
+  <plugin filename="gz-sim-logical-camera-system"
+    name="gz::sim::systems::LogicalCamera">
+  </plugin>
+  <plugin filename="gz-sim-camera-system"
+        name="gz::sim::systems::Camera">
+  </plugin>
   <!-- body link -->
   <gazebo reference="body_link">
     <mu1>0.2</mu1>
     <mu2>0.2</mu2>
-    <material>Gazebo/White</material>
+    <material>
+      <ambient>0.388 0.388 0.388 1</ambient>
+      <diffuse>0.388 0.388 0.388 1</diffuse>
+      <specular>0.388 0.388 0.388 1</specular>
+    </material>
     <selfCollide>false</selfCollide>
   </gazebo>
@@ -42,5 +29,9 @@
     <mu1>0.2</mu1>
     <mu2>0.2</mu2>
-    <material>Gazebo/White</material>
+    <material>
+      <ambient>0.388 0.388 0.388 1</ambient>
+      <diffuse>0.388 0.388 0.388 1</diffuse>
+      <specular>0.388 0.388 0.388 1</specular>
+    </material>
     <selfCollide>false</selfCollide>
   </gazebo>
@@ -48,5 +39,9 @@
     <mu1>0.2</mu1>
     <mu2>0.2</mu2>
-    <material>Gazebo/White</material>
+    <material>
+      <ambient>0.388 0.388 0.388 1</ambient>
+      <diffuse>0.388 0.388 0.388 1</diffuse>
+      <specular>0.388 0.388 0.388 1</specular>
+    </material>
     <selfCollide>false</selfCollide>
   </gazebo>
@@ -54,5 +49,9 @@
     <mu1>0.2</mu1>
     <mu2>0.2</mu2>
-    <material>Gazebo/White</material>
+    <material>
+      <ambient>0.388 0.388 0.388 1</ambient>
+      <diffuse>0.388 0.388 0.388 1</diffuse>
+      <specular>0.388 0.388 0.388 1</specular>
+    </material>
     <selfCollide>false</selfCollide>
   </gazebo>
@@ -60,5 +59,9 @@
     <mu1>0.2</mu1>
     <mu2>0.2</mu2>
-    <material>Gazebo/White</material>
+    <material>
+      <ambient>0.388 0.388 0.388 1</ambient>
+      <diffuse>0.388 0.388 0.388 1</diffuse>
+      <specular>0.388 0.388 0.388 1</specular>
+    </material>
     <selfCollide>false</selfCollide>
   </gazebo>
@@ -66,5 +69,9 @@
     <mu1>0.2</mu1>
     <mu2>0.2</mu2>
-    <material>Gazebo/White</material>
+    <material>
+      <ambient>0.388 0.388 0.388 1</ambient>
+      <diffuse>0.388 0.388 0.388 1</diffuse>
+      <specular>0.388 0.388 0.388 1</specular>
+    </material>
     <selfCollide>false</selfCollide>
   </gazebo>
@@ -77,5 +84,9 @@
     <maxVel>1.0</maxVel>
     <minDepth>0.001</minDepth>
-    <material>Gazebo/White</material>
+    <material>
+      <ambient>0.388 0.388 0.388 1</ambient>
+      <diffuse>0.388 0.388 0.388 1</diffuse>
+      <specular>0.388 0.388 0.388 1</specular>
+    </material>
   </gazebo>
   <!-- right leg links -->
@@ -83,5 +94,9 @@
     <mu1>0.2</mu1>
     <mu2>0.2</mu2>
-    <material>Gazebo/White</material>
+    <material>
+      <ambient>0.388 0.388 0.388 1</ambient>
+      <diffuse>0.388 0.388 0.388 1</diffuse>
+      <specular>0.388 0.388 0.388 1</specular>
+    </material>
     <selfCollide>false</selfCollide>
   </gazebo>
@@ -89,5 +104,9 @@
     <mu1>0.2</mu1>
     <mu2>0.2</mu2>
-    <material>Gazebo/White</material>
+    <material>
+      <ambient>0.388 0.388 0.388 1</ambient>
+      <diffuse>0.388 0.388 0.388 1</diffuse>
+      <specular>0.388 0.388 0.388 1</specular>
+    </material>
     <selfCollide>false</selfCollide>
   </gazebo>
@@ -95,5 +114,9 @@
     <mu1>0.2</mu1>
     <mu2>0.2</mu2>
-    <material>Gazebo/White</material>
+    <material>
+      <ambient>0.388 0.388 0.388 1</ambient>
+      <diffuse>0.388 0.388 0.388 1</diffuse>
+      <specular>0.388 0.388 0.388 1</specular>
+    </material>
     <selfCollide>false</selfCollide>
   </gazebo>
@@ -101,5 +124,9 @@
     <mu1>0.2</mu1>
     <mu2>0.2</mu2>
-    <material>Gazebo/White</material>
+    <material>
+      <ambient>0.388 0.388 0.388 1</ambient>
+      <diffuse>0.388 0.388 0.388 1</diffuse>
+      <specular>0.388 0.388 0.388 1</specular>
+    </material>
     <selfCollide>false</selfCollide>
   </gazebo>
@@ -107,5 +134,9 @@
     <mu1>0.2</mu1>
     <mu2>0.2</mu2>
-    <material>Gazebo/White</material>
+    <material>
+      <ambient>0.388 0.388 0.388 1</ambient>
+      <diffuse>0.388 0.388 0.388 1</diffuse>
+      <specular>0.388 0.388 0.388 1</specular>
+    </material>
     <selfCollide>false</selfCollide>
   </gazebo>
@@ -119,10 +150,18 @@
     <maxVel>1.0</maxVel>
     <minDepth>0.001</minDepth>
-    <material>Gazebo/White</material>
+    <material>
+      <ambient>0.388 0.388 0.388 1</ambient>
+      <diffuse>0.388 0.388 0.388 1</diffuse>
+      <specular>0.388 0.388 0.388 1</specular>
+    </material>
   </gazebo>
   <gazebo reference="r_sho_pitch_link">
     <mu1>0.2</mu1>
     <mu2>0.2</mu2>
-    <material>Gazebo/White</material>
+    <material>
+      <ambient>0.388 0.388 0.388 1</ambient>
+      <diffuse>0.388 0.388 0.388 1</diffuse>
+      <specular>0.388 0.388 0.388 1</specular>
+    </material>
     <selfCollide>false</selfCollide>
   </gazebo>
@@ -130,5 +169,9 @@
     <mu1>0.2</mu1>
     <mu2>0.2</mu2>
-    <material>Gazebo/White</material>
+    <material>
+      <ambient>0.388 0.388 0.388 1</ambient>
+      <diffuse>0.388 0.388 0.388 1</diffuse>
+      <specular>0.388 0.388 0.388 1</specular>
+    </material>
     <selfCollide>false</selfCollide>
   </gazebo>
@@ -136,5 +179,9 @@
     <mu1>0.2</mu1>
     <mu2>0.2</mu2>
-    <material>Gazebo/White</material>
+    <material>
+      <ambient>0.388 0.388 0.388 1</ambient>
+      <diffuse>0.388 0.388 0.388 1</diffuse>
+      <specular>0.388 0.388 0.388 1</specular>
+    </material>
     <selfCollide>false</selfCollide>
   </gazebo>
@@ -142,5 +189,9 @@
     <mu1>0.2</mu1>
     <mu2>0.2</mu2>
-    <material>Gazebo/White</material>
+    <material>
+      <ambient>0.388 0.388 0.388 1</ambient>
+      <diffuse>0.388 0.388 0.388 1</diffuse>
+      <specular>0.388 0.388 0.388 1</specular>
+    </material>
     <selfCollide>false</selfCollide>
   </gazebo>
@@ -148,5 +199,9 @@
     <mu1>0.2</mu1>
     <mu2>0.2</mu2>
-    <material>Gazebo/White</material>
+    <material>
+      <ambient>0.388 0.388 0.388 1</ambient>
+      <diffuse>0.388 0.388 0.388 1</diffuse>
+      <specular>0.388 0.388 0.388 1</specular>
+    </material>
     <selfCollide>false</selfCollide>
   </gazebo>
@@ -154,5 +209,9 @@
     <mu1>0.2</mu1>
     <mu2>0.2</mu2>
-    <material>Gazebo/White</material>
+    <material>
+      <ambient>0.388 0.388 0.388 1</ambient>
+      <diffuse>0.388 0.388 0.388 1</diffuse>
+      <specular>0.388 0.388 0.388 1</specular>
+    </material>
     <selfCollide>false</selfCollide>
   </gazebo>
@@ -160,5 +219,9 @@
     <mu1>0.2</mu1>
     <mu2>0.2</mu2>
-    <material>Gazebo/White</material>
+    <material>
+      <ambient>0.388 0.388 0.388 1</ambient>
+      <diffuse>0.388 0.388 0.388 1</diffuse>
+      <specular>0.388 0.388 0.388 1</specular>
+    </material>
     <selfCollide>false</selfCollide>
   </gazebo>
@@ -166,8 +229,12 @@
     <mu1>0.2</mu1>
     <mu2>0.2</mu2>
-    <material>Gazebo/White</material>
-    <selfCollide>false</selfCollide>
-  </gazebo>
-  <gazebo reference="l_hip_yaw">
+    <material>
+      <ambient>0.388 0.388 0.388 1</ambient>
+      <diffuse>0.388 0.388 0.388 1</diffuse>
+      <specular>0.388 0.388 0.388 1</specular>
+    </material>
+    <selfCollide>false</selfCollide>
+  </gazebo>
+  <!-- <gazebo reference="l_hip_yaw">
     <provideFeedback>1</provideFeedback>
     <implicitSpringDamper>1</implicitSpringDamper>
@@ -248,58 +315,35 @@
     <provideFeedback>1</provideFeedback>
     <implicitSpringDamper>1</implicitSpringDamper>
-  </gazebo>
+  </gazebo> -->
   <!-- head camera -->
-<!--
   <gazebo reference="cam_gazebo_link">
-    <sensor name='camera' type='camera'>
-      <pose>-0.050000 -0.010000 0.000000 -1.5708 0.000000 -3.141592</pose>
-      <camera name='__default__'>
-        <horizontal_fov>1.012300</horizontal_fov>
-        <image>
-          <width>320</width>
-          <height>200</height>
-        </image>
-        <clip>
-          <near>0.001000</near>
-          <far>100.000000</far>
-        </clip>
-      </camera>
-      <always_on>1</always_on>
-      <update_rate>30.000000</update_rate>
-      <visualize>1</visualize>
-      <plugin name="camera_controller" filename="libgazebo_ros_camera.so">
-        <alwaysOn>true</alwaysOn>
-        <updateRate>30</updateRate>
-        <cameraName>robotis_op3/camera</cameraName>
-        <imageTopicName>image_raw</imageTopicName>
-        <cameraInfoTopicName>camera_info</cameraInfoTopicName>
-        <frameName>cam_link</frameName>
-        <hackBaseline>0.07</hackBaseline>
-        <distortionK1>0.0</distortionK1>
-        <distortionK2>0.0</distortionK2>
-        <distortionK3>0.0</distortionK3>
-        <distortionT1>0.0</distortionT1>
-        <distortionT2>0.0</distortionT2>
-      </plugin>
-    </sensor>
-  </gazebo> -->
+    <sensor name="camera" type="camera">
+    <always_on>true</always_on>
+    <visualize>true</visualize>
+    <update_rate>30</update_rate>
+    <topic>gazebo/camera/image_raw</topic>
+    <gz_frame_id>cam_link</gz_frame_id>
+    <camera name="__default__">
+      <camera_info_topic>gazebo/camera/camera_info</camera_info_topic>
+      <horizontal_fov>1.012300</horizontal_fov>
+      <image>
+        <width>320</width>
+        <height>200</height>
+      </image>
+      <clip>
+        <near>0.001000</near>
+        <far>100.000000</far>
+      </clip>
+    </camera>
+  </sensor>
+  </gazebo>
   <!-- imu sensor -->
   <gazebo reference="body_link">
     <gravity>true</gravity>
     <sensor name="imu_sensor" type="imu">
-      <always_on>true</always_on>
-      <update_rate>100</update_rate>
+      <always_on>1</always_on>
+      <update_rate>1</update_rate>
       <visualize>true</visualize>
-      <topic>__default_topic__</topic>
-      <plugin filename="gz-sim-imu-system"
-        name="gz::sim::systems::Imu">
-        <topicName>robotis_op3/imu</topicName>
-        <bodyName>body_link</bodyName>
-        <updateRateHZ>10.0</updateRateHZ>
-        <gaussianNoise>0.0</gaussianNoise>
-        <xyzOffset>0 0 0</xyzOffset>
-        <rpyOffset>0 0 0</rpyOffset>
-        <frameName>body_link</frameName>
-      </plugin>
+      <topic>gazebo/imu</topic>
       <pose>0 0 0 0 0 0</pose>
     </sensor>
