Commit message: change package name to altair_simulation

File: src/altair_simulation/urdf/robotis_op3.urdf.xacro (robot description, xacro)
@@ -1,14 +1,14 @@
 <?xml version="1.0" ?>
 <robot xmlns:xacro="http://www.ros.org/wiki/xacro" name="robotis_op3">
-  <xacro:include filename="$(find op3_description)/urdf/robotis_op3.visuals.xacro" />
-  <xacro:include filename="$(find op3_description)/urdf/robotis_op3.inertia.xacro" />
-  <xacro:include filename="$(find op3_description)/urdf/robotis_op3.structure.rleg.xacro" />
-  <xacro:include filename="$(find op3_description)/urdf/robotis_op3.structure.lleg.xacro" />
-  <xacro:include filename="$(find op3_description)/urdf/robotis_op3.structure.rarm.xacro" />
-  <xacro:include filename="$(find op3_description)/urdf/robotis_op3.structure.larm.xacro" />
-  <xacro:include filename="$(find op3_description)/urdf/robotis_op3.structure.head.xacro" />
-  <xacro:include filename="$(find op3_description)/urdf/robotis_op3.gazebo.xacro" />
-  <!-- <xacro:include filename="$(find op3_description)/urdf/robotis_op3.transmissions.xacro" /> -->
-  <!-- <xacro:include filename="$(find op3_description)/urdf/gazebo_harness.xacro" /> -->
+  <xacro:include filename="$(find altair_simulation)/urdf/robotis_op3.visuals.xacro" />
+  <xacro:include filename="$(find altair_simulation)/urdf/robotis_op3.inertia.xacro" />
+  <xacro:include filename="$(find altair_simulation)/urdf/robotis_op3.structure.rleg.xacro" />
+  <xacro:include filename="$(find altair_simulation)/urdf/robotis_op3.structure.lleg.xacro" />
+  <xacro:include filename="$(find altair_simulation)/urdf/robotis_op3.structure.rarm.xacro" />
+  <xacro:include filename="$(find altair_simulation)/urdf/robotis_op3.structure.larm.xacro" />
+  <xacro:include filename="$(find altair_simulation)/urdf/robotis_op3.structure.head.xacro" />
+  <xacro:include filename="$(find altair_simulation)/urdf/robotis_op3.gazebo.xacro" />
+  <!-- <xacro:include filename="$(find altair_simulation)/urdf/robotis_op3.transmissions.xacro" /> -->
+  <!-- <xacro:include filename="$(find altair_simulation)/urdf/gazebo_harness.xacro" /> -->
   <!-- harness link -->
   <!-- <xacro:add_sim_harness harnessed_link="body_link"/> -->
@@ -34,5 +34,5 @@
     <collision>
       <geometry>
-        <mesh filename="file://$(find op3_description)/meshes/body.stl"  scale="0.001 0.001 0.001"/>
+        <mesh filename="file://$(find altair_simulation)/meshes/body.stl"  scale="0.001 0.001 0.001"/>
       </geometry>
     </collision>

File: src/altair_simulation/urdf/robotis_op3.visuals.xacro (robot description, xacro)
@@ -2,12 +2,12 @@
 <robot xmlns:xacro="http://ros.org/wiki/xacro">
   <!-- <xacro:property name="pi" value="3.141592654" /> -->
-  <!-- file://$(find op3_description) -->
-  <!-- file://$(find op3_description) -->
-  <!-- file://$(find op3_description) -->
+  <!-- file://$(find altair_simulation) -->
+  <!-- file://$(find altair_simulation) -->
+  <!-- file://$(find altair_simulation) -->
   <!-- body link -->
   <xacro:macro name="insert_mesh_body_link">
     <origin xyz="0 0 0" rpy="0 0 0" />
     <geometry>
-      <mesh filename="file://$(find op3_description)/meshes/body.stl"  scale="0.001 0.001 0.001"/>
+      <mesh filename="file://$(find altair_simulation)/meshes/body.stl"  scale="0.001 0.001 0.001"/>
     </geometry>
     <material name="Grey">
@@ -19,5 +19,5 @@
     <origin xyz="0 0 0" rpy="0 0 0" />
     <geometry>
-      <mesh filename="file://$(find op3_description)/meshes/rl1.stl"  scale="0.001 0.001 0.001"/>
+      <mesh filename="file://$(find altair_simulation)/meshes/rl1.stl"  scale="0.001 0.001 0.001"/>
     </geometry>
     <material name="Grey">
@@ -29,5 +29,5 @@
     <origin xyz="0 0 0" rpy="0 0 0" />
     <geometry>
-      <mesh filename="file://$(find op3_description)/meshes/rl2.stl"  scale="0.001 0.001 0.001"/>
+      <mesh filename="file://$(find altair_simulation)/meshes/rl2.stl"  scale="0.001 0.001 0.001"/>
     </geometry>
     <material name="Grey">
@@ -39,5 +39,5 @@
     <origin xyz="0 0 0" rpy="0 0 0" />
     <geometry>
-      <mesh filename="file://$(find op3_description)/meshes/rl3.stl"  scale="0.001 0.001 0.001"/>
+      <mesh filename="file://$(find altair_simulation)/meshes/rl3.stl"  scale="0.001 0.001 0.001"/>
     </geometry>
     <material name="Grey">
@@ -49,5 +49,5 @@
     <origin xyz="0 0 0" rpy="0 0 0" />
     <geometry>
-      <mesh filename="file://$(find op3_description)/meshes/rl4.stl"  scale="0.001 0.001 0.001"/>
+      <mesh filename="file://$(find altair_simulation)/meshes/rl4.stl"  scale="0.001 0.001 0.001"/>
     </geometry>
     <material name="Grey">
@@ -59,5 +59,5 @@
     <origin xyz="0 0 0" rpy="0 0 0" />
     <geometry>
-      <mesh filename="file://$(find op3_description)/meshes/rl5.stl"  scale="0.001 0.001 0.001"/>
+      <mesh filename="file://$(find altair_simulation)/meshes/rl5.stl"  scale="0.001 0.001 0.001"/>
     </geometry>
     <material name="Grey">
@@ -69,5 +69,5 @@
     <origin xyz="0 0 0" rpy="0 0 0" />
     <geometry>
-      <mesh filename="file://$(find op3_description)/meshes/rl6.stl"  scale="0.001 0.001 0.001"/>
+      <mesh filename="file://$(find altair_simulation)/meshes/rl6.stl"  scale="0.001 0.001 0.001"/>
     </geometry>
     <material name="Grey">
@@ -79,5 +79,5 @@
     <origin xyz="0 0 0" rpy="0 0 0" />
     <geometry>
-      <mesh filename="file://$(find op3_description)/meshes/ll1.stl"  scale="0.001 0.001 0.001"/>
+      <mesh filename="file://$(find altair_simulation)/meshes/ll1.stl"  scale="0.001 0.001 0.001"/>
     </geometry>
     <material name="Grey">
@@ -89,5 +89,5 @@
     <origin xyz="0 0 0" rpy="0 0 0" />
     <geometry>
-      <mesh filename="file://$(find op3_description)/meshes/ll2.stl"  scale="0.001 0.001 0.001"/>
+      <mesh filename="file://$(find altair_simulation)/meshes/ll2.stl"  scale="0.001 0.001 0.001"/>
     </geometry>
     <material name="Grey">
@@ -99,5 +99,5 @@
     <origin xyz="0 0 0" rpy="0 0 0" />
     <geometry>
-      <mesh filename="file://$(find op3_description)/meshes/ll3.stl"  scale="0.001 0.001 0.001"/>
+      <mesh filename="file://$(find altair_simulation)/meshes/ll3.stl"  scale="0.001 0.001 0.001"/>
     </geometry>
     <material name="Grey">
@@ -109,5 +109,5 @@
     <origin xyz="0 0 0" rpy="0 0 0" />
     <geometry>
-      <mesh filename="file://$(find op3_description)/meshes/ll4.stl"  scale="0.001 0.001 0.001"/>
+      <mesh filename="file://$(find altair_simulation)/meshes/ll4.stl"  scale="0.001 0.001 0.001"/>
     </geometry>
     <material name="Grey">
@@ -119,5 +119,5 @@
     <origin xyz="0 0 0" rpy="0 0 0" />
     <geometry>
-      <mesh filename="file://$(find op3_description)/meshes/ll5.stl"  scale="0.001 0.001 0.001"/>
+      <mesh filename="file://$(find altair_simulation)/meshes/ll5.stl"  scale="0.001 0.001 0.001"/>
     </geometry>
     <material name="Grey">
@@ -129,5 +129,5 @@
     <origin xyz="0 0 0" rpy="0 0 0" />
     <geometry>
-      <mesh filename="file://$(find op3_description)/meshes/ll6.stl"  scale="0.001 0.001 0.001"/>
+      <mesh filename="file://$(find altair_simulation)/meshes/ll6.stl"  scale="0.001 0.001 0.001"/>
     </geometry>
     <material name="Grey">
@@ -139,5 +139,5 @@
     <origin xyz="0 0 0" rpy="0 0 0" />
     <geometry>
-      <mesh filename="file://$(find op3_description)/meshes/ra1.stl"  scale="0.001 0.001 0.001"/>
+      <mesh filename="file://$(find altair_simulation)/meshes/ra1.stl"  scale="0.001 0.001 0.001"/>
     </geometry>
     <material name="Grey">
@@ -149,5 +149,5 @@
     <origin xyz="0 0 0" rpy="0 0 0" />
     <geometry>
-      <mesh filename="file://$(find op3_description)/meshes/ra2.stl"  scale="0.001 0.001 0.001"/>
+      <mesh filename="file://$(find altair_simulation)/meshes/ra2.stl"  scale="0.001 0.001 0.001"/>
     </geometry>
     <material name="Grey">
@@ -159,5 +159,5 @@
     <origin xyz="0 0 0" rpy="0 0 0" />
     <geometry>
-      <mesh filename="file://$(find op3_description)/meshes/ra3.stl"  scale="0.001 0.001 0.001"/>
+      <mesh filename="file://$(find altair_simulation)/meshes/ra3.stl"  scale="0.001 0.001 0.001"/>
     </geometry>
     <material name="Grey">
@@ -169,5 +169,5 @@
     <origin xyz="0 0 0" rpy="0 0 0" />
     <geometry>
-      <mesh filename="file://$(find op3_description)/meshes/la1.stl"  scale="0.001 0.001 0.001"/>
+      <mesh filename="file://$(find altair_simulation)/meshes/la1.stl"  scale="0.001 0.001 0.001"/>
     </geometry>
     <material name="Grey">
@@ -179,5 +179,5 @@
     <origin xyz="0 0 0" rpy="0 0 0" />
     <geometry>
-      <mesh filename="file://$(find op3_description)/meshes/la2.stl"  scale="0.001 0.001 0.001"/>
+      <mesh filename="file://$(find altair_simulation)/meshes/la2.stl"  scale="0.001 0.001 0.001"/>
     </geometry>
     <material name="Grey">
@@ -189,5 +189,5 @@
     <origin xyz="0 0 0" rpy="0 0 0" />
     <geometry>
-      <mesh filename="file://$(find op3_description)/meshes/la3.stl"  scale="0.001 0.001 0.001"/>
+      <mesh filename="file://$(find altair_simulation)/meshes/la3.stl"  scale="0.001 0.001 0.001"/>
     </geometry>
     <material name="Grey">
@@ -199,5 +199,5 @@
     <origin xyz="0 0 0" rpy="0 0 0" />
     <geometry>
-      <mesh filename="file://$(find op3_description)/meshes/h1.stl"  scale="0.001 0.001 0.001"/>
+      <mesh filename="file://$(find altair_simulation)/meshes/h1.stl"  scale="0.001 0.001 0.001"/>
     </geometry>
     <material name="Grey">
@@ -209,5 +209,5 @@
     <origin xyz="0 0 0" rpy="0 0 0" />
     <geometry>
-      <mesh filename="file://$(find op3_description)/meshes/h2.stl"  scale="0.001 0.001 0.001"/>
+      <mesh filename="file://$(find altair_simulation)/meshes/h2.stl"  scale="0.001 0.001 0.001"/>
     </geometry>
     <material name="Grey">
